File: KiCad Project Files/Swtich Matrix.kicad_sch (KiCad schematic)
At the start: 147 parts

Commit message: QoL Improvements
- Add physical button for Bootloader and Reset.
- Add logic level shifter for the leds according to suggestion by Sleepdealer.
Connections:
- net col0: now also MX5.2 (COL); no longer MX5.1 (COL)
- net at D3.2 (A), MX1.2 (ROW): now also MX5.1 (ROW); no longer MX5.2 (ROW)
Changed lines of the file:
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@@
     (pin "2")
   )
-  (symbol (lib_id "cipulot_parts:MX-LED") (at 36.195 75.565 0) (unit 1)
+  (symbol (lib_name "MX-LED_1") (lib_id "cipulot_parts:MX-LED") (at 36.195 75.565 0) (unit 1)
     (in_bom yes) (on_board yes) (fields_autoplaced)
     (property "Reference" "MX5" (id 0) (at 38.3506 69.215 0)
